File: Power.kicad_sch (KiCad schematic)
At the start: 58 parts, among them J10 VCC, J11 5V, J12 28V, J3 GND, J4 9V, J5 GND, J6 Barrel_Jack_Switch, J8 VPP, J9 GND, Q1 BC327, Q3 BC327, U3 MCP4812, U4 LM358, U6 LM317_TO-220, U7 LD1086V-DG, U8 LM7805_TO220, U9 MC34063AP

Commit message: Minor adjustments
Other:
- note added: "Max current: ~200mA Switching Freq: ~89kHz Vout 1.25(22000/1000+1): 28.75V"
- note removed: "Max current: ~200mA Switching Freq: ~89kHz Vout 1.25(22100/1000+1): 28.75V"
- moved on the sheet: D9
Changed lines of the file:
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@@
 		)
 	)
-	(text "Max current:             ~200mA\nSwitching Freq:          ~89kHz\nVout 1.25(22100/1000+1): 28.75V"
+	(text "Max current:             ~200mA\nSwitching Freq:          ~89kHz\nVout 1.25(22000/1000+1): 28.75V"
 		(exclude_from_sim no)
 		(at 209.55 26.67 0)
@@
 	(wire
 		(pts
-			(xy 125.73 132.08) (xy 125.73 142.24)
+			(xy 125.73 130.81) (xy 125.73 142.24)
 		)
 		(stroke
@@
 	(wire
 		(pts
-			(xy 138.43 132.08) (xy 148.59 132.08)
+			(xy 140.97 130.81) (xy 148.59 130.81)
 		)
 		(stroke
@@
 	(wire
 		(pts
-			(xy 130.81 132.08) (xy 125.73 132.08)
+			(xy 133.35 130.81) (xy 125.73 130.81)
 		)
 		(stroke
@@
 	(wire
 		(pts
-			(xy 148.59 132.08) (xy 148.59 142.24)
+			(xy 148.59 130.81) (xy 148.59 142.24)
 		)
 		(stroke
@@
 	(symbol
 		(lib_id "Diode:B340")
-		(at 134.62 132.08 0)
+		(at 137.16 130.81 0)
 		(unit 1)
 		(exclude_from_sim no)
@@
 		(fields_autoplaced yes)
 		(property "Reference" "D9"
-			(at 134.3025 125.73 0)
+			(at 136.8425 124.46 0)
 			(effects
 				(font
@@
 		)
 		(property "Value" "SB340"
-			(at 134.3025 128.27 0)
+			(at 136.8425 127 0)
 			(effects
 				(font
@@
 		)
 		(property "Footprint" "Diode_THT:D_DO-201AD_P5.08mm_Vertical_KathodeUp"
-			(at 134.62 136.525 0)
+			(at 137.16 135.255 0)
 			(effects
 				(font
@@
 		)
 		(property "Datasheet" "http://www.jameco.com/Jameco/Products/ProdDS/1538777.pdf"
-			(at 134.62 132.08 0)
+			(at 137.16 130.81 0)
 			(effects
 				(font
@@
 		)
 		(property "Description" "40V 3A Schottky Barrier Rectifier Diode, SMC"
-			(at 134.62 132.08 0)
+			(at 137.16 130.81 0)
 			(effects
 				(font
